Commit message: final commit before project submission - full valiation, labelling and testing with some comments

File: TRINA_Model/urdf/TRINA_Defender_v2.urdf (robot description, URDF)
Before this commit: robot Lowpoly_cholera_new_base_URDF_AVATRINA_ver3.0_ECE598_AddedComponentShield, 24 links, 23 joints
Links:
- link base_link: geometry collision mesh filename=./meshes/base_link.STL; visual mesh filename=./meshes/base_link.STL
- link head_base_link: geometry collision mesh filename=./meshes/head_base_link.STL; visual mesh filename=./meshes/head_base_link.STL
- link head_neck1_link: geometry collision mesh filename=./meshes/head_neck1_link.STL; visual mesh filename=./meshes/head_neck1_link.STL
- link head_neck2_link: geometry collision mesh filename=./meshes/head_neck2_link.STL; visual mesh filename=./meshes/head_neck2_link.STL
- link left_EE_link: geometry collision mesh filename=./meshes/left_EE_link.STL; visual mesh filename=./meshes/left_EE_link.STL
- link left_base_link: geometry collision mesh filename=./meshes/left_base_link.STL; visual mesh filename=./meshes/left_base_link.STL
- link left_forearm_link: geometry collision mesh filename=./meshes/left_forearm_link.STL; visual mesh filename=./meshes/left_forearm_link.STL
- link left_shoulder_link: geometry collision mesh filename=./meshes/left_shoulder_link.STL; visual mesh filename=./meshes/left_shoulder_link.STL
- link left_tool_link: geometry collision mesh filename=./meshes/left_tool_link.STL; visual mesh filename=./meshes/left_tool_link.STL
- link left_upperarm_link: geometry collision mesh filename=./meshes/left_upperarm_link.STL; visual mesh filename=./meshes/left_upperarm_link.STL
- link left_wrist1_link: geometry collision mesh filename=./meshes/left_wrist1_link.STL; visual mesh filename=./meshes/left_wrist1_link.STL
- link left_wrist2_camera_link: geometry collision mesh filename=./meshes/left_wrist2_camera_link.STL; visual mesh filename=./meshes/left_wrist2_camera_link.STL
- link left_wrist2_link: geometry collision mesh filename=./meshes/left_wrist2_link.STL; visual mesh filename=./meshes/left_wrist2_link.STL
- link right_EE_link: geometry collision mesh filename=./meshes/right_EE_link.STL; visual mesh filename=./meshes/right_EE_link.STL
- link right_base_link: geometry collision mesh filename=./meshes/right_base_link.STL; visual mesh filename=./meshes/right_base_link.STL
- link right_forearm_link: geometry collision mesh filename=./meshes/right_forearm_link.STL; visual mesh filename=./meshes/right_forearm_link.STL
- link right_shield_link: geometry collision mesh filename=./meshes/right_shield_link.STL; visual mesh filename=./meshes/right_shield_link.STL
- link right_shoulder_link: geometry collision mesh filename=./meshes/right_shoulder_link.STL; visual mesh filename=./meshes/right_shoulder_link.STL
- link right_tool_link: geometry collision mesh filename=./meshes/right_tool_link.STL; visual mesh filename=./meshes/right_tool_link.STL
- link right_upperarm_link: geometry collision mesh filename=./meshes/right_upperarm_link.STL; visual mesh filename=./meshes/right_upperarm_link.STL
- link right_wrist1_link: geometry collision mesh filename=./meshes/right_wrist1_link.STL; visual mesh filename=./meshes/right_wrist1_link.STL
- link right_wrist2_camera_link: geometry collision mesh filename=../meshes/right_wrist2_camera_link.STL; visual mesh filename=../meshes/right_wrist2_camera_link.STL
- link right_wrist2_link: geometry collision mesh filename=./meshes/right_wrist2_link.STL; visual mesh filename=./meshes/right_wrist2_link.STL
- link torso_link: geometry collision mesh filename=./meshes/torso_link.STL; visual mesh filename=./meshes/torso_link.STL
